File: toilet-light.brd (EAGLE design)
At the start: 68.6 x 53.3 mm, 9 parts

Commit message: board for tinkercad — edits
Parts:
- added Lrelay: (no value), AUTODESK_CIRCUITS_BREADBOARD:2P-2.54-65/35MIL
- added P1: 6.2V, AUTODESK_CIRCUITS_BREADBOARD:2P-2.54-65/35MIL
Connections:
- removed net N$1 (its old number): D1.K, D2.K, R3.1, R5.1, U1.GND..
- removed net N$5 (its old number): R5.2, S5.3, U1.2
- new net N$10: R5.2, S5.2, U1.2
- new net N$6: D1.K, D2.K, Lrelay.2, R3.1, R5.1, U1.GND..
- new net N$7: P1.2, U1.VIN
- new net N$9: R3.2, S1.2, U1.3
- net N$4: now also Lrelay.1, S1.3, S5.3; no longer S1.2, S5.2
- net N$8: now also P1.1, U1.GND.; no longer R3.2, S1.3, U1.3
Changed lines of the file:
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@@
 </autorouter>
 <elements>
-<element value="" name="U1" library="AUTODESK_CIRCUITS_BREADBOARD" package="ARDUINO_UNO" x="5" y="10.08"></element><element value="" name="D1" library="AUTODESK_CIRCUITS_BREADBOARD" package="LED5MM" x="5" y="22.78"></element><element value="" name="D2" library="AUTODESK_CIRCUITS_BREADBOARD" package="LED5MM" x="5" y="35.480000000000004"></element><element value="1k‎Ω" name="R2" library="AUTODESK_CIRCUITS_BREADBOARD" package="0207/10" x="5" y="48.18"></element><element value="1k‎Ω" name="R1" library="AUTODESK_CIRCUITS_BREADBOARD" package="0207/10" x="5" y="60.879999999999995"></element><element value="10k‎Ω" name="R3" library="AUTODESK_CIRCUITS_BREADBOARD" package="0207/10" x="5" y="73.58"></element><element value="10k‎Ω" name="R5" library="AUTODESK_CIRCUITS_BREADBOARD" package="0207/10" x="5" y="86.28"></element><element value="" name="S5" library="AUTODESK_CIRCUITS_BREADBOARD" package="M251" x="5" y="98.98"></element><element value="" name="S1" library="AUTODESK_CIRCUITS_BREADBOARD" package="M251" x="5" y="111.68"></element></elements>
+<element value="" name="U1" library="AUTODESK_CIRCUITS_BREADBOARD" package="ARDUINO_UNO" x="5" y="10.08"></element><element value="" name="D1" library="AUTODESK_CIRCUITS_BREADBOARD" package="LED5MM" x="5" y="22.78"></element><element value="" name="D2" library="AUTODESK_CIRCUITS_BREADBOARD" package="LED5MM" x="5" y="35.480000000000004"></element><element value="1k‎Ω" name="R2" library="AUTODESK_CIRCUITS_BREADBOARD" package="0207/10" x="5" y="48.18"></element><element value="1k‎Ω" name="R1" library="AUTODESK_CIRCUITS_BREADBOARD" package="0207/10" x="5" y="60.879999999999995"></element><element value="10k‎Ω" name="R3" library="AUTODESK_CIRCUITS_BREADBOARD" package="0207/10" x="5" y="73.58"></element><element value="10k‎Ω" name="R5" library="AUTODESK_CIRCUITS_BREADBOARD" package="0207/10" x="5" y="86.28"></element><element value="" name="S5" library="AUTODESK_CIRCUITS_BREADBOARD" package="M251" x="5" y="98.98"></element><element value="" name="S1" library="AUTODESK_CIRCUITS_BREADBOARD" package="M251" x="5" y="111.68"></element><element value="" name="Lrelay" library="AUTODESK_CIRCUITS_BREADBOARD" package="2P-2.54-65/35MIL" x="5" y="124.38000000000001"></element><element value="6.2V" name="P1" library="AUTODESK_CIRCUITS_BREADBOARD" package="2P-2.54-65/35MIL" x="5" y="137.08"></element></elements>
 <signals>
-<signal name="N$1"><contactref element="R5" pad="1"></contactref><contactref element="D1" pad="K"></contactref><wire x1="-0.08000000000000007" y1="86.28" x2="6.27" y2="22.78" width="0" layer="19" extent="1-1"></wire><contactref element="D2" pad="K"></contactref><wire x1="6.27" y1="22.78" x2="6.27" y2="35.480000000000004" width="0" layer="19" extent="1-1"></wire><contactref element="U1" pad="GND.."></contactref><wire x1="6.27" y1="35.480000000000004" x2="45.64" y2="12.620000000000001" width="0" layer="19" extent="1-1"></wire><contactref element="R3" pad="1"></contactref><wire x1="45.64" y1="12.620000000000001" x2="-0.08000000000000007" y2="73.58" width="0" layer="19" extent="1-1"></wire></signal><signal name="N$2"><contactref element="U1" pad="7"></contactref><contactref element="R1" pad="2"></contactref><wire x1="50.72" y1="60.879999999999995" x2="10.08" y2="60.879999999999995" width="0" layer="19" extent="1-1"></wire></signal><signal name="N$3"><contactref element="R2" pad="2"></contactref><contactref element="U1" pad="4"></contactref><wire x1="10.08" y1="48.18" x2="58.34" y2="60.879999999999995" width="0" layer="19" extent="1-1"></wire></signal><signal name="N$4"><contactref element="S5" pad="2"></contactref><contactref element="U1" pad="5V"></contactref><wire x1="5" y1="98.98" x2="43.1" y2="12.620000000000001" width="0" layer="19" extent="1-1"></wire><contactref element="S1" pad="2"></contactref><wire x1="43.1" y1="12.620000000000001" x2="5" y2="111.68" width="0" layer="19" extent="1-1"></wire></signal><signal name="N$5"><contactref element="R5" pad="2"></contactref><contactref element="U1" pad="2"></contactref><wire x1="10.08" y1="86.28" x2="63.42" y2="60.879999999999995" width="0" layer="19" extent="1-1"></wire><contactref element="S5" pad="3"></contactref><wire x1="63.42" y1="60.879999999999995" x2="7.54" y2="98.98" width="0" layer="19" extent="1-1"></wire></signal><signal name="N$6"><contactref element="R1" pad="1"></contactref><contactref element="D1" pad="A"></contactref><wire x1="-0.08000000000000007" y1="60.879999999999995" x2="3.73" y2="22.78" width="0" layer="19" extent="1-1"></wire></signal><signal name="N$7"><contactref element="R2" pad="1"></contactref><contactref element="D2" pad="A"></contactref><wire x1="-0.08000000000000007" y1="48.18" x2="3.73" y2="35.480000000000004" width="0" layer="19" extent="1-1"></wire></signal><signal name="N$8"><contactref element="U1" pad="3"></contactref><contactref element="S1" pad="3"></contactref><wire x1="60.88" y1="60.879999999999995" x2="7.54" y2="111.68" width="0" layer="19" extent="1-1"></wire><contactref element="R3" pad="2"></contactref><wire x1="7.54" y1="111.68" x2="10.08" y2="73.58" width="0" layer="19" extent="1-1"></wire></signal></signals>
+<signal name="N$1"><contactref element="R1" pad="2"></contactref><contactref element="U1" pad="7"></contactref><wire x1="10.08" y1="60.879999999999995" x2="50.72" y2="60.879999999999995" width="0" layer="19" extent="1-1"></wire></signal><signal name="N$2"><contactref element="D1" pad="A"></contactref><contactref element="R1" pad="1"></contactref><wire x1="3.73" y1="22.78" x2="-0.08000000000000007" y2="60.879999999999995" width="0" layer="19" extent="1-1"></wire></signal><signal name="N$3"><contactref element="D2" pad="A"></contactref><contactref element="R2" pad="1"></contactref><wire x1="3.73" y1="35.480000000000004" x2="-0.08000000000000007" y2="48.18" width="0" layer="19" extent="1-1"></wire></signal><signal name="N$4"><contactref element="S1" pad="3"></contactref><contactref element="U1" pad="5V"></contactref><wire x1="7.54" y1="111.68" x2="43.1" y2="12.620000000000001" width="0" layer="19" extent="1-1"></wire><contactref element="Lrelay" pad="1"></contactref><wire x1="43.1" y1="12.620000000000001" x2="5" y2="125.65" width="0" layer="19" extent="1-1"></wire><contactref element="S5" pad="3"></contactref><wire x1="5" y1="125.65" x2="7.54" y2="98.98" width="0" layer="19" extent="1-1"></wire></signal><signal name="N$5"><contactref element="U1" pad="4"></contactref><contactref element="R2" pad="2"></contactref><wire x1="58.34" y1="60.879999999999995" x2="10.08" y2="48.18" width="0" layer="19" extent="1-1"></wire></signal><signal name="N$6"><contactref element="U1" pad="GND.."></contactref><contactref element="R5" pad="1"></contactref><wire x1="45.64" y1="12.620000000000001" x2="-0.08000000000000007" y2="86.28" width="0" layer="19" extent="1-1"></wire><contactref element="R3" pad="1"></contactref><wire x1="-0.08000000000000007" y1="86.28" x2="-0.08000000000000007" y2="73.58" width="0" layer="19" extent="1-1"></wire><contactref element="D2" pad="K"></contactref><wire x1="-0.08000000000000007" y1="73.58" x2="6.27" y2="35.480000000000004" width="0" layer="19" extent="1-1"></wire><contactref element="D1" pad="K"></contactref><wire x1="6.27" y1="35.480000000000004" x2="6.27" y2="22.78" width="0" layer="19" extent="1-1"></wire><contactref element="Lrelay" pad="2"></contactref><wire x1="6.27" y1="22.78" x2="5" y2="123.11000000000001" width="0" layer="19" extent="1-1"></wire></signal><signal name="N$7"><contactref element="P1" pad="2"></contactref><contactref element="U1" pad="VIN"></contactref><wire x1="5" y1="135.81" x2="50.72" y2="12.620000000000001" width="0" layer="19" extent="1-1"></wire></signal><signal name="N$8"><contactref element="P1" pad="1"></contactref><contactref element="U1" pad="GND."></contactref><wire x1="5" y1="138.35000000000002" x2="48.18" y2="12.620000000000001" width="0" layer="19" extent="1-1"></wire></signal><signal name="N$9"><contactref element="U1" pad="3"></contactref><contactref element="S1" pad="2"></contactref><wire x1="60.88" y1="60.879999999999995" x2="5" y2="111.68" width="0" layer="19" extent="1-1"></wire><contactref element="R3" pad="2"></contactref><wire x1="5" y1="111.68" x2="10.08" y2="73.58" width="0" layer="19" extent="1-1"></wire></signal><signal name="N$10"><contactref element="S5" pad="2"></contactref><contactref element="U1" pad="2"></contactref><wire x1="5" y1="98.98" x2="63.42" y2="60.879999999999995" width="0" layer="19" extent="1-1"></wire><contactref element="R5" pad="2"></contactref><wire x1="63.42" y1="60.879999999999995" x2="10.08" y2="86.28" width="0" layer="19" extent="1-1"></wire></signal></signals>
 </board>
 </drawing>
